Commit message: new file:   build/dronut_description/build/lib/dronut_description/move.py 	modified:   build/dronut_description/colcon_command_prefix_setup_py.sh.env 	modified:   build/dronut_description/dronut_description.egg-info/SOURCES.txt 	modified:   build/dronut_description/dronut_description.egg-info/entry_points.txt 	modified:   build/dronut_description/install.log 	modified:   build/dronut_description/prefix_override/__pycache__/sitecustomize.cpython-310.pyc 	new file:   install/dronut_description/lib/dronut_description/move 	modified:   install/dronut_description/lib/python3.10/site-packages/dronut_description-0.0.0-py3.10.egg-info/SOURCES.txt 	modified:   install/dronut_description/lib/python3.10/site-packages/dronut_description-0.0.0-py3.10.egg-info/entry_points.txt 	new file:   install/dronut_description/lib/python3.10/site-packages/dronut_description/__pycache__/move.cpython-310.pyc 	new file:   install/dronut_description/lib/python3.10/site-packages/dronut_description/move.py 	modified:   install/dronut_description/share/dronut_description/launch/__pycache__/drone.launch.cpython-310.pyc 	modified:   install/dronut_description/share/dronut_description/launch/drone.launch.py 	modified:   install/dronut_description/share/dronut_description/urdf/x1.urdf.xacro 	new file:   log/build_2024-12-20_11-30-08/dronut_description/command.log 	new file:   log/build_2024-12-20_11-30-08/dronut_description/stderr.log 	new file:   log/build_2024-12-20_11-30-08/dronut_description/stdout.log 	new file:   log/build_2024-12-20_11-30-08/dronut_description/stdout_stderr.log 	new file:   log/build_2024-12-20_11-30-08/dronut_description/streams.log 	new file:   log/build_2024-12-20_11-30-08/events.log 	new file:   log/build_2024-12-20_11-30-08/logger_all.log 	new file:   log/build_2024-12-20_11-37-06/dronut_description/command.log 	new file:   log/build_2024-12-20_11-37-06/dronut_description/stderr.log 	new file:   log/build_2024-12-20_11-37-06/dronut_description/stdout.log 	new file:   log/build_2024-12-20_11-37-06/dronut_description/stdout_stderr.log 	new file:   log/build_2024-12-20_11-37-06/dronut_description/streams.log 	new file:   log/build_2024-12-20_11-37-06/events.log 	new file:   log/build_2024-12-20_11-37-06/logger_all.log 	modified:   log/latest_build 	new file:   src/dronut_description/dronut_description/move.py 	modified:   src/dronut_description/launch/drone.launch.py 	modified:   src/dronut_description/setup.py 	modified:   src/dronut_description/urdf/x1.urdf.xacro

File: install/dronut_description/share/dronut_description/urdf/x1.urdf.xacro (robot description, xacro)
@@ -466,5 +466,5 @@
 </inertial>
 </link>
-<joint name="slider1" type="prismatic">
+<joint name="slider_front" type="prismatic">
 <origin xyz="1.2347761702002914081e-16 -8.6977309035618530899e-17 0.022430000000000005489" rpy="-2.2551405187698405946e-17 -4.770489558936214117e-18 1.570796326794896558" />
 <parent link="part_9" />
@@ -496,5 +496,5 @@
 </inertial>
 </link>
-<joint name="slider2" type="prismatic">
+<joint name="slider_back" type="prismatic">
 <origin xyz="6.2776311926526772165e-17 2.0448052973076597602e-17 0.036080000000000014837" rpy="2.6454533008646252723e-17 5.6378512969245521826e-18 2.2954338760707362899e-16" />
 <parent link="part_9" />
@@ -526,5 +526,5 @@
 </inertial>
 </link>
-<joint name="slider3" type="prismatic">
+<joint name="slider_left" type="prismatic">
 <origin xyz="7.3121474153392539981e-17 -2.0789429205914076587e-17 0.022160000000000006082" rpy="-4.3368086899420129212e-19 -2.3418766925686846471e-17 4.5622041572063771955e-17" />
 <parent link="part_9" />
@@ -556,5 +556,5 @@
 </inertial>
 </link>
-<joint name="slider4" type="prismatic">
+<joint name="slider_right" type="prismatic">
 <origin xyz="8.0144224590128492692e-17 -2.1194452443085178714e-17 0.056060000000000012599" rpy="2.2551405187698396701e-17 8.6736173798847114735e-19 -1.570796326794896558" />
 <parent link="part_9" />
