Commit message: renamed:    install/dronut_description/lib/python3.10/site-packages/dronut_description/__init__.py -> build/dronut_controller/.cmake/api/v1/query/client-colcon-cmake/codemodel-v2 	new file:   build/dronut_controller/.cmake/api/v1/reply/codemodel-v2-04302853cd162e523f20.json 	new file:   build/dronut_controller/.cmake/api/v1/reply/directory-.-ede247d097fb88cd60bc.json 	new file:   build/dronut_controller/.cmake/api/v1/reply/index-2024-12-24T20-47-48-0134.json 	new file:   build/dronut_controller/.cmake/api/v1/reply/target-drone_control_node-46f71ab5b0ef3620ca34.json 	new file:   build/dronut_controller/.cmake/api/v1/reply/target-dronut_controller_uninstall-ae7d195e5fb9e65a9be2.json 	new file:   build/dronut_controller/.cmake/api/v1/reply/target-uninstall-c8e3cfb4cbf8b38191d2.json 	renamed:    log/build_2024-12-19_16-56-40/dronut_description/stderr.log -> build/dronut_controller/AMENT_IGNORE 	new file:   build/dronut_controller/CMakeCache.txt 	new file:   build/dronut_controller/CMakeFiles/3.28.3/CMakeCCompiler.cmake 	new file:   build/dronut_controller/CMakeFiles/3.28.3/CMakeCXXCompiler.cmake 	new file:   build/dronut_controller/CMakeFiles/3.28.3/CMakeDetermineCompilerABI_C.bin 	new file:   build/dronut_controller/CMakeFiles/3.28.3/CMakeDetermineCompilerABI_CXX.bin 	new file:   build/dronut_controller/CMakeFiles/3.28.3/CMakeSystem.cmake 	new file:   build/dronut_controller/CMakeFiles/3.28.3/CompilerIdC/CMakeCCompilerId.c 	new file:   build/dronut_controller/CMakeFiles/3.28.3/CompilerIdC/a.out 	new file:   build/dronut_controller/CMakeFiles/3.28.3/CompilerIdCXX/CMakeCXXCompilerId.cpp 	new file:   build/dronut_controller/CMakeFiles/3.28.3/CompilerIdCXX/a.out 	new file:   build/dronut_controller/CMakeFiles/CMakeConfigureLog.yaml 	new file:   build/dronut_controller/CMakeFiles/CMakeDirectoryInformation.cmake 	new file:   build/dronut_controller/CMakeFiles/CMakeRuleHashes.txt 	new file:   build/dronut_controller/CMakeFiles/Makefile.cmake 	new file:   build/dronut_controller/CMakeFiles/Makefile2 	new file:   build/dronut_controller/CMakeFiles/TargetDirectories.txt 	new file:   build/dronut_controller/CMakeFiles/cmake.check_cache 	new file:   build/dronut_controller/CMakeFiles/drone_control_node.dir/DependInfo.cmake 	new file:   build/dronut_controller/CMakeFiles/drone_control_node.dir/build.make 	new file:   build/dronut_controller/CMakeFiles/drone_control_node.dir/cmake_clean.cmake 	new file:   build/dronut_controller/CMakeFiles/drone_control_node.dir/compiler_depend.internal 	new file:   build/dronut_controller/CMakeFiles/drone_control_node.dir/compiler_depend.make 	new file:   build/dronut_controller/CMakeFiles/drone_control_node.dir/compiler_depend.ts 	new file:   build/dronut_controller/CMakeFiles/drone_control_node.dir/depend.make 	new file:   build/dronut_controller/CMakeFiles/drone_control_node.dir/flags.make 	new file:   build/dronut_controller/CMakeFiles/drone_control_node.dir/link.txt 	new file:   build/dronut_controller/CMakeFiles/drone_control_node.dir/progress.make 	new file:   build/dronut_controller/CMakeFiles/drone_control_node.dir/src/birotor_drone_controller.cpp.o 	new file:   build/dronut_controller/CMakeFiles/drone_control_node.dir/src/birotor_drone_controller.cpp.o.d 	new file:   build/dronut_controller/CMakeFiles/drone_control_node.dir/src/joy_to_cmd_vel_node.cpp.o 	new file:   build/dronut_controller/CMakeFiles/drone_control_node.dir/src/joy_to_cmd_vel_node.cpp.o.d 	new file:   build/dronut_controller/CMakeFiles/drone_control_node.dir/src/main.cpp.o 	new file:   build/dronut_controller/CMakeFiles/drone_control_node.dir/src/main.cpp.o.d 	new file:   build/dronut_controller/CMakeFiles/dronut_controller_uninstall.dir/DependInfo.cmake 	new file:   build/dronut_controller/CMakeFiles/dronut_controller_uninstall.dir/build.make 	new file:   build/dronut_controller/CMakeFiles/dronut_controller_uninstall.dir/cmake_clean.cmake 	new file:   build/dronut_controller/CMakeFiles/dronut_controller_uninstall.dir/compiler_depend.make 	new file:   build/dronut_controller/CMakeFiles/dronut_controller_uninstall.dir/compiler_depend.ts 	renamed:    install/dronut_description/lib/python3.10/site-packages/dronut_description-0.0.0-py3.10.egg-info/dependency_links.txt -> build/dronut_controller/CMakeFiles/dronut_controller_uninstall.dir/progress.make 	new file:   build/dronut_controller/CMakeFiles/progress.marks 	new file:   build/dronut_controller/CMakeFiles/uninstall.dir/DependInfo.cmake 	new file:   build/dronut_controller/CMakeFiles/uninstall.dir/build.make 	new file:   build/dronut_controller/CMakeFiles/uninstall.dir/cmake_clean.cmake 	new file:   build/dronut_controller/CMakeFiles/uninstall.dir/compiler_depend.make 	new file:   build/dronut_controller/CMakeFiles/uninstall.dir/compiler_depend.ts 	renamed:    install/dronut_description/lib/python3.10/site-packages/dronut_description-0.0.0-py3.10.egg-info/zip-safe -> build/dronut_controller/CMakeFiles/uninstall.dir/progress.make 	new file:   build/dronut_controller/CTestConfiguration.ini 	new file:   build/dronut_controller/CTestCustom.cmake 	new file:   build/dronut_controller/CTestTestfile.cmake 	new file:   build/dronut_controller/Makefile 	new file:   build/dronut_controller/ament_cmake_core/dronut_controllerConfig-version.cmake 	new file:   build/dronut_controller/ament_cmake_core/dronut_controllerConfig.cmake 	new file:   build/dronut_controller/ament_cmake_core/package.cmake 	new file:   build/dronut_controller/ament_cmake_core/stamps/ament_prefix_path.sh.stamp 	new file:   build/dronut_controller/ament_cmake_core/stamps/nameConfig-version.cmake.in.stamp 	new file:   build/dronut_controller/ament_cmake_core/stamps/nameConfig.cmake.in.stamp 	new file:   build/dronut_controller/ament_cmake_core/stamps/package.xml.stamp 	new file:   build/dronut_controller/ament_cmake_core/stamps/package_xml_2_cmake.py.stamp 	new file:   build/dronut_controller/ament_cmake_core/stamps/path.sh.stamp 	new file:   build/dronut_controller/ament_cmake_core/stamps/templates_2_cmake.py.stamp 	new file:   build/dronut_controller/ament_cmake_environment_hooks/ament_prefix_path.dsv 	new file:   build/dronut_controller/ament_cmake_environment_hooks/local_setup.bash 	new file:   build/dronut_controller/ament_cmake_environment_hooks/local_setup.dsv 	new file:   build/dronut_controller/ament_cmake_environment_hooks/local_setup.sh 	new file:   build/dronut_controller/ament_cmake_environment_hooks/local_setup.zsh 	new file:   build/dronut_controller/ament_cmake_environment_hooks/package.dsv 	new file:   build/dronut_controller/ament_cmake_environment_hooks/path.dsv 	new file:   build/dronut_controller/ament_cmake_index/share/ament_index/resource_index/package_run_dependencies/dronut_controller 	renamed:    log/build_2024-12-19_17-00-03/dronut_description/stderr.log -> build/dronut_controller/ament_cmake_index/share/ament_index/resource_index/packages/dronut_controller 	new file:   build/dronut_controller/ament_cmake_index/share/ament_index/resource_index/parent_prefix_path/dronut_controller 	new file:   build/dronut_controller/ament_cmake_package_templates/templates.cmake 	new file:   build/dronut_controller/ament_cmake_uninstall_target/ament_cmake_uninstall_target.cmake 	new file:   build/dronut_controller/cmake_args.last 	new file:   build/dronut_controller/cmake_install.cmake 	new file:   build/dronut_controller/colcon_build.rc 	new file:   build/dronut_controller/colcon_command_prefix_build.sh 	new file:   build/dronut_controller/colcon_command_prefix_build.sh.env 	new file:   build/dronut_controller/drone_control_node 	new file:   build/dronut_controller/install_manifest.txt 	modified:   build/dronut_description/build/lib/dronut_description/move.py 	modified:   build/dronut_description/colcon_command_prefix_setup_py.sh.env 	modified:   build/dronut_description/dronut_description.egg-info/PKG-INFO 	modified:   build/dronut_description/dronut_description.egg-info/entry_points.txt 	modified:   build/dronut_description/install.log 	deleted:    build/dronut_description/prefix_override/__pycache__/sitecustomize.cpython-310.pyc 	new file:   build/dronut_description/prefix_override/__pycache__/sitecustomize.cpython-312.pyc 	renamed:    log/build_2024-12-19_17-00-35/dronut_description/stderr.log -> build/dronut_w_cam/build/lib/dronut_w_cam/__init__.py 	renamed:    install/dronut_description/lib/python3.10/site-packages/dronut_description/move.py -> build/dronut_w_cam/build/lib/dronut_w_cam/move.py 	new file:   build/dronut_w_cam/colcon_build.rc 	new file:   build/dronut_w_cam/colcon_command_prefix_setup_py.sh 	new file:   build/dronut_w_cam/colcon_command_prefix_setup_py.sh.env 	renamed:    install/dronut_description/lib/python3.10/site-packages/dronut_description-0.0.0-py3.10.egg-info/PKG-INFO -> build/dronut_w_cam/dronut_w_cam.egg-info/PKG-INFO 	new file:   build/dronut_w_cam/dronut_w_cam.egg-info/SOURCES.txt 	new file:   build/dronut_w_cam/dronut_w_cam.egg-info/dependency_links.txt 	new file:   build/dronut_w_cam/dronut_w_cam.egg-info/entry_points.txt 	renamed:    install/dronut_description/lib/python3.10/site-packages/dronut_description-0.0.0-py3.10.egg-info/requires.txt -> build/dronut_w_cam/dronut_w_cam.egg-info/requires.txt 	new file:   build/dronut_w_cam/dronut_w_cam.egg-info/top_level.txt 	new file:   build/dronut_w_cam/dronut_w_cam.egg-info/zip-safe 	new file:   build/dronut_w_cam/install.log 	new file:   build/dronut_w_cam/prefix_override/__pycache__/sitecustomize.cpython-312.pyc 	new file:   build/dronut_w_cam/prefix_override/sitecustomize.py 	renamed:    log/build_2024-12-19_17-14-36/dronut_description/stderr.log -> build/joy_test/.cmake/api/v1/query/client-colcon-cmake/codemodel-v2 	new file:   build/joy_test/.cmake/api/v1/reply/codemodel-v2-5054d9a6e5af77300756.json 	new file:   build/joy_test/.cmake/api/v1/reply/directory-.-0e9e7bcb71e88cae72b6.json 	new file:   build/joy_test/.cmake/api/v1/reply/index-2024-12-24T20-46-53-0041.json 	new file:   build/joy_test/.cmake/api/v1/reply/target-joy_test_node-3ef8dd1c0c1a1cfa4eeb.json 	new file:   build/joy_test/.cmake/api/v1/reply/target-joy_test_uninstall-cd48741698055ae473c3.json 	new file:   build/joy_test/.cmake/api/v1/reply/target-uninstall-fc47768189cf6b2273c9.json 	renamed:    log/build_2024-12-20_11-30-08/dronut_description/stderr.log -> build/joy_test/AMENT_IGNORE 	new file:   build/joy_test/CMakeCache.txt 	new file:   build/joy_test/CMakeFiles/3.28.3/CMakeCCompiler.cmake 	new file:   build/joy_test/CMakeFiles/3.28.3/CMakeCXXCompiler.cmake 	new file:   build/joy_test/CMakeFiles/3.28.3/CMakeDetermineCompilerABI_C.bin 	new file:   build/joy_test/CMakeFiles/3.28.3/CMakeDetermineCompilerABI_CXX.bin 	new file:   build/joy_test/CMakeFiles/3.28.3/CMakeSystem.cmake 	new file:   build/joy_test/CMakeFiles/3.28.3/CompilerIdC/CMakeCCompilerId.c 	new file:   build/joy_test/CMakeFiles/3.28.3/CompilerIdC/a.out 	new file:   build/joy_test/CMakeFiles/3.28.3/CompilerIdCXX/CMakeCXXCompilerId.cpp 	new file:   build/joy_test/CMakeFiles/3.28.3/CompilerIdCXX/a.out 	new file:   build/joy_test/CMakeFiles/CMakeConfigureLog.yaml 	new file:   build/joy_test/CMakeFiles/CMakeDirectoryInformation.cmake 	new file:   build/joy_test/CMakeFiles/CMakeRuleHashes.txt 	new file:   build/joy_test/CMakeFiles/Makefile.cmake 	new file:   build/joy_test/CMakeFiles/Makefile2 	new file:   build/joy_test/CMakeFiles/TargetDirectories.txt 	new file:   build/joy_test/CMakeFiles/cmake.check_cache 	new file:   build/joy_test/CMakeFiles/joy_test_node.dir/DependInfo.cmake 	new file:   build/joy_test/CMakeFiles/joy_test_node.dir/build.make 	new file:   build/joy_test/CMakeFiles/joy_test_node.dir/cmake_clean.cmake 	new file:   build/joy_test/CMakeFiles/joy_test_node.dir/compiler_depend.internal 	new file:   build/joy_test/CMakeFiles/joy_test_node.dir/compiler_depend.make 	new file:   build/joy_test/CMakeFiles/joy_test_node.dir/compiler_depend.ts 	new file:   build/joy_test/CMakeFiles/joy_test_node.dir/depend.make 	new file:   build/joy_test/CMakeFiles/joy_test_node.dir/flags.make 	new file:   build/joy_test/CMakeFiles/joy_test_node.dir/link.txt 	new file:   build/joy_test/CMakeFiles/joy_test_node.dir/progress.make 	new file:   build/joy_test/CMakeFiles/joy_test_node.dir/src/joy.cpp.o 	new file:   build/joy_test/CMakeFiles/joy_test_node.dir/src/joy.cpp.o.d 	new file:   build/joy_test/CMakeFiles/joy_test_uninstall.dir/DependInfo.cmake 	new file:   build/joy_test/CMakeFiles/joy_test_uninstall.dir/build.make 	new file:   build/joy_test/CMakeFiles/joy_test_uninstall.dir/cmake_clean.cmake 	new file:   build/joy_test/CMakeFiles/joy_test_uninstall.dir/compiler_depend.make 	new file:   build/joy_test/CMakeFiles/joy_test_uninstall.dir/compiler_depend.ts 	new file:   build/joy_test/CMakeFiles/joy_test_uninstall.dir/progress.make 	new file:   build/joy_test/CMakeFiles/progress.marks 	new file:   build/joy_test/CMakeFiles/uninstall.dir/DependInfo.cmake 	new file:   build/joy_test/CMakeFiles/uninstall.dir/build.make 	new file:   build/joy_test/CMakeFiles/uninstall.dir/cmake_clean.cmake 	new file:   build/joy_test/CMakeFiles/uninstall.dir/compiler_depend.make 	new file:   build/joy_test/CMakeFiles/uninstall.dir/compiler_depend.ts 	new file:   build/joy_test/CMakeFiles/uninstall.dir/progress.make 	new file:   build/joy_test/CTestConfiguration.ini 	new file:   build/joy_test/CTestCustom.cmake 	new file:   build/joy_test/CTestTestfile.cmake 	new file:   build/joy_test/Makefile 	new file:   build/joy_test/ament_cmake_core/joy_testConfig-version.cmake 	new file:   build/joy_test/ament_cmake_core/joy_testConfig.cmake 	new file:   build/joy_test/ament_cmake_core/package.cmake 	new file:   build/joy_test/ament_cmake_core/stamps/ament_prefix_path.sh.stamp 	new file:   build/joy_test/ament_cmake_core/stamps/nameConfig-version.cmake.in.stamp 	new file:   build/joy_test/ament_cmake_core/stamps/nameConfig.cmake.in.stamp 	new file:   build/joy_test/ament_cmake_core/stamps/package.xml.stamp 	new file:   build/joy_test/ament_cmake_core/stamps/package_xml_2_cmake.py.stamp 	new file:   build/joy_test/ament_cmake_core/stamps/path.sh.stamp 	new file:   build/joy_test/ament_cmake_core/stamps/templates_2_cmake.py.stamp 	new file:   build/joy_test/ament_cmake_environment_hooks/ament_prefix_path.dsv 	new file:   build/joy_test/ament_cmake_environment_hooks/local_setup.bash 	new file:   build/joy_test/ament_cmake_environment_hooks/local_setup.dsv 	new file:   build/joy_test/ament_cmake_environment_hooks/local_setup.sh 	new file:   build/joy_test/ament_cmake_environment_hooks/local_setup.zsh 	new file:   build/joy_test/ament_cmake_environment_hooks/package.dsv 	new file:   build/joy_test/ament_cmake_environment_hooks/path.dsv 	new file:   build/joy_test/ament_cmake_index/share/ament_index/resource_index/package_run_dependencies/joy_test 	renamed:    log/build_2024-12-20_11-37-06/dronut_description/stderr.log -> build/joy_test/ament_cmake_index/share/ament_index/resource_index/packages/joy_test 	new file:   build/joy_test/ament_cmake_index/share/ament_index/resource_index/parent_prefix_path/joy_test 	new file:   build/joy_test/ament_cmake_package_templates/templates.cmake 	new file:   build/joy_test/ament_cmake_uninstall_target/ament_cmake_uninstall_target.cmake 	new file:   build/joy_test/cmake_args.last 	new file:   build/joy_test/cmake_install.cmake 	new file:   build/joy_test/colcon_build.rc 	new file:   build/joy_test/colcon_command_prefix_build.sh 	new file:   build/joy_test/colcon_command_prefix_build.sh.env 	new file:   build/joy_test/install_manifest.txt 	new file:   build/joy_test/joy_test_node 	new file:   build/realsense_cam/build/lib/realsense_cam/__init__.py 	new file:   build/realsense_cam/colcon_build.rc 	new file:   build/realsense_cam/colcon_command_prefix_setup_py.sh 	new file:   build/realsense_cam/colcon_command_prefix_setup_py.sh.env 	new file:   build/realsense_cam/install.log 	new file:   build/realsense_cam/prefix_override/__pycache__/sitecustomize.cpython-312.pyc 	new file:   build/realsense_cam/prefix_override/sitecustomize.py 	new file:   build/realsense_cam/realsense_cam.egg-info/PKG-INFO 	new file:   build/realsense_cam/realsense_cam.egg-info/SOURCES.txt 	new file:   build/realsense_cam/realsense_cam.egg-info/dependency_links.txt 	new file:   build/realsense_cam/realsense_cam.egg-info/requires.txt 	new file:   build/realsense_cam/realsense_cam.egg-info/top_level.txt 	new file:   build/realsense_cam/realsense_cam.egg-info/zip-safe 	new file:   install/dronut_controller/lib/dronut_controller/drone_control_node 	new file:   install/dronut_controller/share/ament_index/resource_index/package_run_dependencies/dronut_controller 	new file:   install/dronut_controller/share/ament_index/resource_index/packages/dronut_controller 	new file:   install/dronut_controller/share/ament_index/resource_index/parent_prefix_path/dronut_controller 	new file:   install/dronut_controller/share/colcon-core/packages/dronut_controller 	new file:   install/dronut_controller/share/dronut_controller/cmake/dronut_controllerConfig-version.cmake 	new file:   install/dronut_controller/share/dronut_controller/cmake/dronut_controllerConfig.cmake 	new file:   install/dronut_controller/share/dronut_controller/environment/ament_prefix_path.dsv 	new file:   install/dronut_controller/share/dronut_controller/environment/ament_prefix_path.sh 	new file:   install/dronut_controller/share/dronut_controller/environment/path.dsv 	new file:   install/dronut_controller/share/dronut_controller/environment/path.sh 	new file:   install/dronut_controller/share/dronut_controller/hook/cmake_prefix_path.dsv 	new file:   install/dronut_controller/share/dronut_controller/hook/cmake_prefix_path.ps1 	new file:   install/dronut_controller/share/dronut_controller/hook/cmake_prefix_path.sh 	new file:   install/dronut_controller/share/dronut_controller/launch/__pycache__/drone.launch.cpython-312.pyc 	new file:   install/dronut_controller/share/dronut_controller/launch/drone.launch.py 	new file:   install/dronut_controller/share/dronut_controller/local_setup.bash 	new file:   install/dronut_controller/share/dronut_controller/local_setup.dsv 	new file:   install/dronut_controller/share/dronut_controller/local_setup.sh 	new file:   install/dronut_controller/share/dronut_controller/local_setup.zsh 	new file:   install/dronut_controller/share/dronut_controller/package.bash 	new file:   install/dronut_controller/share/dronut_controller/package.dsv 	new file:   install/dronut_controller/share/dronut_controller/package.ps1 	new file:   install/dronut_controller/share/dronut_controller/package.sh 	new file:   install/dronut_controller/share/dronut_controller/package.xml 	new file:   install/dronut_controller/share/dronut_controller/package.zsh 	deleted:    install/dronut_description/lib/python3.10/site-packages/dronut_description/__pycache__/__init__.cpython-310.pyc 	deleted:    install/dronut_description/lib/python3.10/site-packages/dronut_description/__pycache__/move.cpython-310.pyc 	new file:   install/dronut_description/lib/python3.12/site-packages/dronut_description-0.0.0-py3.12.egg-info/PKG-INFO 	renamed:    install/dronut_description/lib/python3.10/site-packages/dronut_description-0.0.0-py3.10.egg-info/SOURCES.txt -> install/dronut_description/lib/python3.12/site-packages/dronut_description-0.0.0-py3.12.egg-info/SOURCES.txt 	new file:   install/dronut_description/lib/python3.12/site-packages/dronut_description-0.0.0-py3.12.egg-info/dependency_links.txt 	renamed:    install/dronut_description/lib/python3.10/site-packages/dronut_description-0.0.0-py3.10.egg-info/entry_points.txt -> install/dronut_description/lib/python3.12/site-packages/dronut_description-0.0.0-py3.12.egg-info/entry_points.txt 	new file:   install/dronut_description/lib/python3.12/site-packages/dronut_description-0.0.0-py3.12.egg-info/requires.txt 	renamed:    install/dronut_description/lib/python3.10/site-packages/dronut_description-0.0.0-py3.10.egg-info/top_level.txt -> install/dronut_description/lib/pyt

File: install/dronut_description/share/dronut_description/urdf/x1.urdf.xacro (robot description, xacro)
@@ -2,4 +2,9 @@
 <robot xmlns:xacro="http://www.ros.org/wiki/xacro" name="dronut">
 <xacro:include filename="$(find dronut_description)/urdf/x1.gazebo.xacro"/>
+<link name="base_link">
+    <visual>
+    <origin xyz="0 0 0" rpy="0 0 ${3.141592653589793/4}"/>
+    </visual>
+</link>
 <link name="part_9">
 <visual>
@@ -24,4 +29,10 @@
 </inertial>
 </link>
+<joint name="base_link_part9" type="fixed">
+    <origin xyz="0 0 0" rpy="0 0 0"/>
+    <parent link="base_link" />
+    <child link="part_9" />
+    <axis xyz="0 0 1"/>
+</joint>
 <link name="part_14">
 <visual>
