Commit message: renamed:    build/dronut_controller/.cmake/api/v1/reply/codemodel-v2-04302853cd162e523f20.json -> build/dronut_controller/.cmake/api/v1/reply/codemodel-v2-bf6b74380779ce25cd13.json 	renamed:    build/dronut_controller/.cmake/api/v1/reply/directory-.-ede247d097fb88cd60bc.json -> build/dronut_controller/.cmake/api/v1/reply/directory-.-3a44757d298d8532200f.json 	renamed:    build/dronut_controller/.cmake/api/v1/reply/index-2024-12-24T20-47-48-0134.json -> build/dronut_controller/.cmake/api/v1/reply/index-2025-01-06T16-05-41-0561.json 	renamed:    build/dronut_controller/.cmake/api/v1/reply/target-drone_control_node-46f71ab5b0ef3620ca34.json -> build/dronut_controller/.cmake/api/v1/reply/target-drone_control_node-17b52511751b96ea8097.json 	modified:   build/dronut_controller/CMakeCache.txt 	modified:   build/dronut_controller/CMakeFiles/CMakeConfigureLog.yaml 	modified:   build/dronut_controller/CMakeFiles/Makefile.cmake 	modified:   build/dronut_controller/CMakeFiles/drone_control_node.dir/build.make 	modified:   build/dronut_controller/CMakeFiles/drone_control_node.dir/compiler_depend.internal 	modified:   build/dronut_controller/CMakeFiles/drone_control_node.dir/compiler_depend.make 	modified:   build/dronut_controller/CMakeFiles/drone_control_node.dir/flags.make 	modified:   build/dronut_controller/CMakeFiles/drone_control_node.dir/link.txt 	modified:   build/dronut_controller/CMakeFiles/drone_control_node.dir/src/birotor_drone_controller.cpp.o 	modified:   build/dronut_controller/CMakeFiles/drone_control_node.dir/src/birotor_drone_controller.cpp.o.d 	modified:   build/dronut_controller/CMakeFiles/drone_control_node.dir/src/joy_to_cmd_vel_node.cpp.o 	modified:   build/dronut_controller/CMakeFiles/drone_control_node.dir/src/joy_to_cmd_vel_node.cpp.o.d 	modified:   build/dronut_controller/CMakeFiles/drone_control_node.dir/src/main.cpp.o 	modified:   build/dronut_controller/CMakeFiles/drone_control_node.dir/src/main.cpp.o.d 	new file:   build/dronut_controller/CMakeFiles/drone_control_node.dir/src/trial_code.cpp.o 	new file:   build/dronut_controller/CMakeFiles/drone_control_node.dir/src/trial_code.cpp.o.d 	modified:   build/dronut_controller/CTestTestfile.cmake 	modified:   build/dronut_controller/ament_cmake_index/share/ament_index/resource_index/parent_prefix_path/dronut_controller 	modified:   build/dronut_controller/cmake_install.cmake 	modified:   build/dronut_controller/colcon_command_prefix_build.sh.env 	modified:   build/dronut_controller/drone_control_node 	modified:   build/dronut_controller/install_manifest.txt 	modified:   build/dronut_description/colcon_command_prefix_setup_py.sh.env 	modified:   build/dronut_description/prefix_override/__pycache__/sitecustomize.cpython-312.pyc 	modified:   build/dronut_w_cam/colcon_command_prefix_setup_py.sh.env 	modified:   build/dronut_w_cam/prefix_override/__pycache__/sitecustomize.cpython-312.pyc 	renamed:    build/joy_test/.cmake/api/v1/reply/codemodel-v2-5054d9a6e5af77300756.json -> build/joy_test/.cmake/api/v1/reply/codemodel-v2-c5f5c3981344ada0556c.json 	renamed:    build/joy_test/.cmake/api/v1/reply/index-2024-12-24T20-46-53-0041.json -> build/joy_test/.cmake/api/v1/reply/index-2025-01-06T16-39-34-0031.json 	renamed:    build/joy_test/.cmake/api/v1/reply/target-joy_test_node-3ef8dd1c0c1a1cfa4eeb.json -> build/joy_test/.cmake/api/v1/reply/target-joy_test_node-f898503088fd3007742a.json 	modified:   build/joy_test/CMakeFiles/Makefile.cmake 	modified:   build/joy_test/CMakeFiles/joy_test_node.dir/build.make 	modified:   build/joy_test/CMakeFiles/joy_test_node.dir/compiler_depend.internal 	modified:   build/joy_test/CMakeFiles/joy_test_node.dir/compiler_depend.make 	modified:   build/joy_test/CMakeFiles/joy_test_node.dir/link.txt 	modified:   build/joy_test/CMakeFiles/joy_test_node.dir/src/joy.cpp.o 	modified:   build/joy_test/CMakeFiles/joy_test_node.dir/src/joy.cpp.o.d 	modified:   build/joy_test/ament_cmake_index/share/ament_index/resource_index/parent_prefix_path/joy_test 	modified:   build/joy_test/colcon_command_prefix_build.sh.env 	modified:   build/joy_test/joy_test_node 	modified:   build/realsense_cam/colcon_command_prefix_setup_py.sh.env 	modified:   build/realsense_cam/prefix_override/__pycache__/sitecustomize.cpython-312.pyc 	modified:   install/dronut_controller/lib/dronut_controller/drone_control_node 	modified:   install/dronut_controller/share/ament_index/resource_index/parent_prefix_path/dronut_controller 	new file:   install/dronut_controller/share/dronut_controller/config/dronut_controllers.yaml 	modified:   install/dronut_controller/share/dronut_controller/launch/__pycache__/drone.launch.cpython-312.pyc 	modified:   install/dronut_controller/share/dronut_controller/launch/drone.launch.py 	new file:   install/dronut_controller/share/dronut_controller/worlds/.sample.jpg 	new file:   install/dronut_controller/share/dronut_controller/worlds/empty.sdf 	new file:   install/dronut_controller/share/dronut_controller/worlds/maze1.sdf 	new file:   install/dronut_controller/share/dronut_controller/worlds/sample.wbt 	new file:   install/dronut_controller/share/dronut_controller/worlds/trial.sdf 	new file:   install/dronut_description/share/dronut_description/launch/__pycache__/drone.launch.cpython-312.pyc 	new file:   install/dronut_description/share/dronut_description/launch/__pycache__/drone_sim.launch.cpython-312.pyc 	new file:   install/dronut_w_cam/share/dronut_w_cam/launch/__pycache__/drone.launch.cpython-312.pyc 	new file:   install/dronut_w_cam/share/dronut_w_cam/launch/__pycache__/drone_sim.launch.cpython-312.pyc 	modified:   install/dronut_w_cam/share/dronut_w_cam/package.xml 	modified:   install/dronut_w_cam/share/dronut_w_cam/rviz/x1_view.rviz 	modified:   install/dronut_w_cam/share/dronut_w_cam/urdf/x1.urdf.xacro 	modified:   install/joy_test/lib/joy_test/joy_test_node 	modified:   install/joy_test/share/ament_index/resource_index/parent_prefix_path/joy_test 	new file:   install/realsense_cam/share/realsense_cam/launch/__pycache__/depth.launch.cpython-312.pyc 	modified:   install/setup.bash 	modified:   install/setup.ps1 	modified:   install/setup.sh 	modified:   install/setup.zsh 	new file:   log/build_2024-12-24_22-00-30/dronut_controller/command.log 	new file:   log/build_2024-12-24_22-00-30/dronut_controller/stderr.log 	new file:   log/build_2024-12-24_22-00-30/dronut_controller/stdout.log 	new file:   log/build_2024-12-24_22-00-30/dronut_controller/stdout_stderr.log 	new file:   log/build_2024-12-24_22-00-30/dronut_controller/streams.log 	new file:   log/build_2024-12-24_22-00-30/dronut_w_cam/command.log 	new file:   log/build_2024-12-24_22-00-30/dronut_w_cam/stderr.log 	new file:   log/build_2024-12-24_22-00-30/dronut_w_cam/stdout.log 	new file:   log/build_2024-12-24_22-00-30/dronut_w_cam/stdout_stderr.log 	new file:   log/build_2024-12-24_22-00-30/dronut_w_cam/streams.log 	new file:   log/build_2024-12-24_22-00-30/events.log 	new file:   log/build_2024-12-24_22-00-30/logger_all.log 	new file:   log/build_2024-12-24_22-02-35/dronut_controller/command.log 	new file:   log/build_2024-12-24_22-02-35/dronut_controller/stderr.log 	new file:   log/build_2024-12-24_22-02-35/dronut_controller/stdout.log 	new file:   log/build_2024-12-24_22-02-35/dronut_controller/stdout_stderr.log 	new file:   log/build_2024-12-24_22-02-35/dronut_controller/streams.log 	new file:   log/build_2024-12-24_22-02-35/dronut_w_cam/command.log 	new file:   log/build_2024-12-24_22-02-35/dronut_w_cam/stderr.log 	new file:   log/build_2024-12-24_22-02-35/dronut_w_cam/stdout.log 	new file:   log/build_2024-12-24_22-02-35/dronut_w_cam/stdout_stderr.log 	new file:   log/build_2024-12-24_22-02-35/dronut_w_cam/streams.log 	new file:   log/build_2024-12-24_22-02-35/events.log 	new file:   log/build_2024-12-24_22-02-35/logger_all.log 	new file:   log/build_2024-12-24_22-06-14/dronut_controller/command.log 	new file:   log/build_2024-12-24_22-06-14/dronut_controller/stderr.log 	new file:   log/build_2024-12-24_22-06-14/dronut_controller/stdout.log 	new file:   log/build_2024-12-24_22-06-14/dronut_controller/stdout_stderr.log 	new file:   log/build_2024-12-24_22-06-14/dronut_controller/streams.log 	new file:   log/build_2024-12-24_22-06-14/dronut_w_cam/command.log 	new file:   log/build_2024-12-24_22-06-14/dronut_w_cam/stderr.log 	new file:   log/build_2024-12-24_22-06-14/dronut_w_cam/stdout.log 	new file:   log/build_2024-12-24_22-06-14/dronut_w_cam/stdout_stderr.log 	new file:   log/build_2024-12-24_22-06-14/dronut_w_cam/streams.log 	new file:   log/build_2024-12-24_22-06-14/events.log 	new file:   log/build_2024-12-24_22-06-14/logger_all.log 	new file:   log/build_2024-12-24_22-11-45/dronut_controller/command.log 	new file:   log/build_2024-12-24_22-11-45/dronut_controller/stderr.log 	new file:   log/build_2024-12-24_22-11-45/dronut_controller/stdout.log 	new file:   log/build_2024-12-24_22-11-45/dronut_controller/stdout_stderr.log 	new file:   log/build_2024-12-24_22-11-45/dronut_controller/streams.log 	new file:   log/build_2024-12-24_22-11-45/dronut_w_cam/command.log 	new file:   log/build_2024-12-24_22-11-45/dronut_w_cam/stderr.log 	new file:   log/build_2024-12-24_22-11-45/dronut_w_cam/stdout.log 	new file:   log/build_2024-12-24_22-11-45/dronut_w_cam/stdout_stderr.log 	new file:   log/build_2024-12-24_22-11-45/dronut_w_cam/streams.log 	new file:   log/build_2024-12-24_22-11-45/events.log 	new file:   log/build_2024-12-24_22-11-45/logger_all.log 	new file:   log/build_2024-12-24_22-13-03/dronut_controller/command.log 	new file:   log/build_2024-12-24_22-13-03/dronut_controller/stderr.log 	new file:   log/build_2024-12-24_22-13-03/dronut_controller/stdout.log 	new file:   log/build_2024-12-24_22-13-03/dronut_controller/stdout_stderr.log 	new file:   log/build_2024-12-24_22-13-03/dronut_controller/streams.log 	new file:   log/build_2024-12-24_22-13-03/dronut_w_cam/command.log 	new file:   log/build_2024-12-24_22-13-03/dronut_w_cam/stderr.log 	new file:   log/build_2024-12-24_22-13-03/dronut_w_cam/stdout.log 	new file:   log/build_2024-12-24_22-13-03/dronut_w_cam/stdout_stderr.log 	new file:   log/build_2024-12-24_22-13-03/dronut_w_cam/streams.log 	new file:   log/build_2024-12-24_22-13-03/events.log 	new file:   log/build_2024-12-24_22-13-03/logger_all.log 	new file:   log/build_2024-12-24_23-28-25/dronut_controller/command.log 	new file:   log/build_2024-12-24_23-28-25/dronut_controller/stderr.log 	new file:   log/build_2024-12-24_23-28-25/dronut_controller/stdout.log 	new file:   log/build_2024-12-24_23-28-25/dronut_controller/stdout_stderr.log 	new file:   log/build_2024-12-24_23-28-25/dronut_controller/streams.log 	new file:   log/build_2024-12-24_23-28-25/events.log 	new file:   log/build_2024-12-24_23-28-25/logger_all.log 	new file:   log/build_2024-12-24_23-28-42/dronut_controller/command.log 	new file:   log/build_2024-12-24_23-28-42/dronut_controller/stderr.log 	new file:   log/build_2024-12-24_23-28-42/dronut_controller/stdout.log 	new file:   log/build_2024-12-24_23-28-42/dronut_controller/stdout_stderr.log 	new file:   log/build_2024-12-24_23-28-42/dronut_controller/streams.log 	new file:   log/build_2024-12-24_23-28-42/events.log 	new file:   log/build_2024-12-24_23-28-42/logger_all.log 	new file:   log/build_2024-12-24_23-28-52/dronut_controller/command.log 	new file:   log/build_2024-12-24_23-28-52/dronut_controller/stderr.log 	new file:   log/build_2024-12-24_23-28-52/dronut_controller/stdout.log 	new file:   log/build_2024-12-24_23-28-52/dronut_controller/stdout_stderr.log 	new file:   log/build_2024-12-24_23-28-52/dronut_controller/streams.log 	new file:   log/build_2024-12-24_23-28-52/events.log 	new file:   log/build_2024-12-24_23-28-52/logger_all.log 	new file:   log/build_2024-12-24_23-29-03/dronut_controller/command.log 	new file:   log/build_2024-12-24_23-29-03/dronut_controller/stderr.log 	new file:   log/build_2024-12-24_23-29-03/dronut_controller/stdout.log 	new file:   log/build_2024-12-24_23-29-03/dronut_controller/stdout_stderr.log 	new file:   log/build_2024-12-24_23-29-03/dronut_controller/streams.log 	new file:   log/build_2024-12-24_23-29-03/events.log 	new file:   log/build_2024-12-24_23-29-03/logger_all.log 	new file:   log/build_2024-12-24_23-29-20/dronut_controller/command.log 	new file:   log/build_2024-12-24_23-29-20/dronut_controller/stderr.log 	new file:   log/build_2024-12-24_23-29-20/dronut_controller/stdout.log 	new file:   log/build_2024-12-24_23-29-20/dronut_controller/stdout_stderr.log 	new file:   log/build_2024-12-24_23-29-20/dronut_controller/streams.log 	new file:   log/build_2024-12-24_23-29-20/events.log 	new file:   log/build_2024-12-24_23-29-20/logger_all.log 	new file:   log/build_2024-12-24_23-29-30/dronut_controller/command.log 	new file:   log/build_2024-12-24_23-29-30/dronut_controller/stderr.log 	new file:   log/build_2024-12-24_23-29-30/dronut_controller/stdout.log 	new file:   log/build_2024-12-24_23-29-30/dronut_controller/stdout_stderr.log 	new file:   log/build_2024-12-24_23-29-30/dronut_controller/streams.log 	new file:   log/build_2024-12-24_23-29-30/events.log 	new file:   log/build_2024-12-24_23-29-30/logger_all.log 	new file:   log/build_2024-12-24_23-30-28/dronut_controller/command.log 	new file:   log/build_2024-12-24_23-30-28/dronut_controller/stderr.log 	new file:   log/build_2024-12-24_23-30-28/dronut_controller/stdout.log 	new file:   log/build_2024-12-24_23-30-28/dronut_controller/stdout_stderr.log 	new file:   log/build_2024-12-24_23-30-28/dronut_controller/streams.log 	new file:   log/build_2024-12-24_23-30-28/events.log 	new file:   log/build_2024-12-24_23-30-28/logger_all.log 	new file:   log/build_2024-12-25_00-07-03/dronut_controller/command.log 	new file:   log/build_2024-12-25_00-07-03/dronut_controller/stderr.log 	new file:   log/build_2024-12-25_00-07-03/dronut_controller/stdout.log 	new file:   log/build_2024-12-25_00-07-03/dronut_controller/stdout_stderr.log 	new file:   log/build_2024-12-25_00-07-03/dronut_controller/streams.log 	new file:   log/build_2024-12-25_00-07-03/events.log 	new file:   log/build_2024-12-25_00-07-03/logger_all.log 	new file:   log/build_2024-12-25_00-09-16/dronut_controller/command.log 	new file:   log/build_2024-12-25_00-09-16/dronut_controller/stderr.log 	new file:   log/build_2024-12-25_00-09-16/dronut_controller/stdout.log 	new file:   log/build_2024-12-25_00-09-16/dronut_controller/stdout_stderr.log 	new file:   log/build_2024-12-25_00-09-16/dronut_controller/streams.log 	new file:   log/build_2024-12-25_00-09-16/dronut_w_cam/command.log 	new file:   log/build_2024-12-25_00-09-16/dronut_w_cam/stderr.log 	new file:   log/build_2024-12-25_00-09-16/dronut_w_cam/stdout.log 	new file:   log/build_2024-12-25_00-09-16/dronut_w_cam/stdout_stderr.log 	new file:   log/build_2024-12-25_00-09-16/dronut_w_cam/streams.log 	new file:   log/build_2024-12-25_00-09-16/events.log 	new file:   log/build_2024-12-25_00-09-16/logger_all.log 	new file:   log/build_2024-12-25_00-14-13/dronut_controller/command.log 	new file:   log/build_2024-12-25_00-14-13/dronut_controller/stderr.log 	new file:   log/build_2024-12-25_00-14-13/dronut_controller/stdout.log 	new file:   log/build_2024-12-25_00-14-13/dronut_controller/stdout_stderr.log 	new file:   log/build_2024-12-25_00-14-13/dronut_controller/streams.log 	new file:   log/build_2024-12-25_00-14-13/dronut_w_cam/command.log 	new file:   log/build_2024-12-25_00-14-13/dronut_w_cam/stderr.log 	new file:   log/build_2024-12-25_00-14-13/dronut_w_cam/stdout.log 	new file:   log/build_2024-12-25_00-14-13/dronut_w_cam/stdout_stderr.log 	new file:   log/build_2024-12-25_00-14-13/dronut_w_cam/streams.log 	new file:   log/build_2024-12-25_00-14-13/events.log 	new file:   log/build_2024-12-25_00-14-13/logger_all.log 	new file:   log/build_2024-12-25_00-16-53/dronut_controller/command.log 	new file:   log/build_2024-12-25_00-16-53/dronut_controller/stderr.log 	new file:   log/build_2024-12-25_00-16-53/dronut_controller/stdout.log 	new file:   log/build_2024-12-25_00-16-53/dronut_controller/stdout_stderr.log 	new file:   log/build_2024-12-25_00-16-53/dronut_controller/streams.log 	new file:   log/build_2024-12-25_00-16-53/dronut_w_cam/command.log 	new file:   log/build_2024-12-25_00-16-53/dronut_w_cam/stderr.log 	new file:   log/build_2024-12-25_00-16-53/dronut_w_cam/stdout.log 	new file:   log/build_2024-12-25_00-16-53/dronut_w_cam/stdout_stderr.log 	new file:   log/build_2024-12-25_00-16-53/dronut_w_cam/streams.log 	new file:   log/build_2024-12-25_00-16-53/events.log 	new file:   log/build_2024-12-25_00-16-53/logger_all.log 	new file:   log/build_2024-12-25_00-20-03/dronut_controller/command.log 	new file:   log/build_2024-12-25_00-20-03/dronut_controller/stderr.log 	new file:   log/build_2024-12-25_00-20-03/dronut_controller/stdout.log 	new file:   log/build_2024-12-25_00-20-03/dronut_controller/stdout_stderr.log 	new file:   log/build_2024-12-25_00-20-03/dronut_controller/streams.log 	new file:   log/build_2024-12-25_00-20-03/dronut_w_cam/command.log 	new file:   log/build_2024-12-25_00-20-03/dronut_w_cam/stderr.log 	new file:   log/build_2024-12-25_00-20-03/dronut_w_cam/stdout.log 	new file:   log/build_2024-12-25_00-20-03/dronut_w_cam/stdout_stderr.log 	new file:   log/build_2024-12-25_00-20-03/dronut_w_cam/streams.log 	new file:   log/build_2024-12-25_00-20-03/events.log 	new file:   log/build_2024-12-25_00-20-03/logger_all.log 	new file:   log/build_2024-12-25_00-32-28/dronut_controller/command.log 	new file:   log/build_2024-12-25_00-32-28/dronut_controller/stderr.log 	new file:   log/build_2024-12-25_00-32-28/dronut_controller/stdout.log 	new file:   log/build_2024-12-25_00-32-28/dronut_controller/stdout_stderr.log 	new file:   log/build_2024-12-25_00-32-28/dronut_controller/streams.log 	new file:   log/build_2024-12-25_00-32-28/dronut_w_cam/command.log 	new file:   log/build_2024-12-25_00-32-28/dronut_w_cam/stderr.log 	new file:   log/build_2024-12-25_00-32-28/dronut_w_cam/stdout.log 	new file:   log/build_2024-12-25_00-32-28/dronut_w_cam/stdout_stderr.log 	new file:   log/build_2024-12-25_00-32-28/dronut_w_cam/streams.log 	new file:   log/build_2024-12-25_00-32-28/events.log 	new file:   log/build_2024-12-25_00-32-28/logger_all.log 	new file:   log/build_2024-12-25_01-05-15/dronut_controller/command.log 	new file:   log/build_2024-12-25_01-05-15/dronut_controller/stderr.log 	new file:   log/build_2024-12-25_01-05-15/dronut_controller/stdout.log 	new file:   log/build_2024-12-25_01-05-15/dronut_controller/stdout_stderr.log 	new file:   log/build_2024-12-25_01-05-15/dronut_controller/streams.log 	new file:   log/build_2024-12-25_01-05-15/dronut_w_cam/command.log 	new file:   log/build_2024-12-25_01-05-15/dronut_w_cam/stderr.log 	new file:   log/build_2024-12-25_01-05-15/dronut_w_cam/stdout.log 	new file:   log/build_2024-12-25_01-05-15/dronut_w_cam/stdout_stderr.log 	new file:   log/build_2024-12-25_01-05-15/dronut_w_cam/streams.log 	new file:   log/build_2024-12-25_01-05-15/events.log 	new file:   log/build_2024-12-25_01-05-15/logger_all.log 	new file:   log/build_2024-12-25_01-10-58/dronut_controller/command.log 	new file:   log/build_2024-12-25_01-10-58/dronut_controller/stderr.log 	new file:   log/build_2024-12-25_01-10-58/dronut_controller/stdout.log 	new file:   log/build_2024-12-25_01-10-58/dronut_controller/stdout_stderr.log 	new file:   log/build_2024-12-25_01-10-58/dronut_controller/streams.log 	new file:   log/build_2024-12-25_01-10-58/dronut_w_cam/command.log 	new file:   log/build_2024-12-25_01-10-58/dronut_w_cam/stderr.log 	new file:   log/build_2024-12-25_01-10-58/dronut_w_cam/stdout.log 	new file:   log/build_2024-12-25_01-10-58/dronut_w_cam/stdout_stderr.log 	new file:   log/build_2024-12-25_01-10-58/dronut_w_cam/streams.log 	new file:   log/build_2024-12-25_01-10-58/events.log 	new file:   log/build_2024-12-25_01-10-58/logger_all.log 	new file:   log/build_2024-12-25_16-26-48/dronut_controller/command.log 	new file:

File: src/dronut_w_cam/urdf/x1.urdf.xacro (robot description, xacro)
@@ -2,9 +2,4 @@
 <robot xmlns:xacro="http://www.ros.org/wiki/xacro" name="dronut">
 <xacro:include filename="$(find realsense_cam)/urdf/test_d455_camera.urdf.xacro"/>
-<link name="base_link">
-    <visual>
-    <origin xyz="0 0 0" rpy="0 0 ${3.141592653589793/4}"/>
-    </visual>
-</link>
 <link name="part_9">
 <visual>
@@ -29,10 +24,4 @@
 </inertial>
 </link>
-<joint name="base_link_part9" type="fixed">
-    <origin xyz="0 0 0" rpy="0 0 0"/>
-    <parent link="base_link" />
-    <child link="part_9" />
-    <axis xyz="0 0 1"/>
-</joint>
 <link name="part_14">
 <visual>
@@ -581,10 +570,73 @@
     <axis xyz="0 0 1"/>
 </joint>
+<gazebo reference="camera_link">
+    <sensor name="rgbd_camera" type="rgbd_camera">
+      <camera>
+        <horizontal_fov>1.25</horizontal_fov>
+        <image>
+          <width>320</width>
+          <height>240</height>
+        </image>
+        <clip>
+          <near>0.3</near>
+          <far>15</far>
+        </clip>
+            <optical_frame_id>camera_infra1_optical_frame</optical_frame_id>
+      </camera>
+      <always_on>1</always_on>
+      <update_rate>20</update_rate>
+      <visualize>true</visualize>
+      <topic>camera</topic>
+      <gz_frame_id>camera_link</gz_frame_id>
+    </sensor>
+  </gazebo>
+<ros2_control name="dronut" type="system">
+    <hardware>
+        <plugin>gz_ros2_control/GazeboSimSystem</plugin>
+    </hardware>
+    <joint name="bottom_prop_continuous">
+        <command_interface name="position"/>
+        <state_interface name="position"/>
+    </joint>
+    <joint name="top_prop_continuous">
+        <command_interface name="position"/>
+        <state_interface name="position"/>
+    </joint>
+    <joint name="slider_front">
+        <command_interface name="position">
+            <param name="min">0.015</param>
+            <param name="max">0.041</param>
+        </command_interface>
+        <state_interface name="position"/>
+    </joint>
+    <joint name="slider_back">
+        <command_interface name="position">
+            <param name="min">-0.019</param>
+            <param name="max">0.008</param>
+        </command_interface>
+        <state_interface name="position"/>
+    </joint>
+    <joint name="slider_left">
+        <command_interface name="position">
+            <param name="min">0.015</param>
+            <param name="max">0.041</param>
+        </command_interface>
+        <state_interface name="position"/>
+    </joint>
+    <joint name="slider_right">
+        <command_interface name="position">
+            <param name="min">-0.018</param>
+            <param name="max">0.009</param>
+        </command_interface>
+        <state_interface name="position"/>
+    </joint>
+</ros2_control>
 <gazebo>
-    <plugin name="gazebo_ros_control" filename="libgazebo_ros_control.so">
-        <robotNamespace>/dronut</robotNamespace>
-        <tf_topic>/model/dronut/tf</tf_topic>
+    <plugin filename="libgz_ros2_control-system" name="gz_ros2_control::GazeboSimROS2ControlPlugin">
+        <parameters>$(find dronut_controller)/config/dronut_controllers.yaml</parameters>
+            <ros>
+                <remapping>/controller_manager/robot_description:=/robot_description</remapping>
+            </ros>
     </plugin>
-    <plugin name="gazebo_ros" filename="libgazebo_ros_api_plugin.so"/>
 </gazebo>
 </robot>
